File: hardware/pcb/iamaerial/iamaerial.kicad_sch (KiCad schematic)
At the start: 65 parts, among them J1 USB_C_Receptacle, J10 USART2_PINOUT, J11 I2C2_PINOUT, J2 ELRS, J3 ESC1, J4 ESC1, J5 ESC1, J6 ESC1, J7 STM32_STLINK, J8 SPI3_PINOUT, J9 USART4_PINOUT, SW1 SW_SPDT, U1 STM32F722RETx, U2 USBLC6-2SC6, U3 ICM-42688-P, U4 DPS368XTSA1, U5 MP2451DJ-LF-Z, U6 AP2112K-3.3TRG1, U7 W25Q128JVSIQ, Y1 ASE-25MHz

Commit message: fix: checked major components on fc with ds, fixed oscillator and made minor adjustments to other smds
Parts:
- removed C10, C11: 20pF, symbol Device:C
- added C25: 1uF, symbol Device:C
- added J12: XT_WIRE_SOLDERING_HOLES, symbol Connector:Conn_01x02_Socket
- C18: value 4.7nF -> 4.7uF
- U4: DESCRIPTION Package dimensions: 8-pin LGA, 2.0 x 2.5 x 1.1 mm3 | Operat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 -> (none)
Connections:
- net VDDIO_BARO is gone; now on net +3.3V: R4.2, R5.2
- net +3.3V: now also C12.2, C13.2, C14.2, C15.2, C16.2, C18.2, C20.2, C21.2, C22.2, C23.2, C24.2, D1.2 (A), D2.1 (K), D5.1 (K), D6.1 (K), J1.A1 (GND), J1.A12 (GND), J1.B1 (GND), J1.B12 (GND), J1.S1 (SHIELD), J2.4 (Pin_4), J7.5 (Pin_5), LS1.N, R13.1, R2.2, R3.2, R6.1, SW1.1 (A), U1.12 (VSSA), U1.18 (VSS), U1.31 (VSS), U1.47 (VSS), U1.63 (VSS), U2.2 (GND), U3.11 (RESV_11), U3.6 (GND), U3.9 (INT2/FSYNC/CLKIN), U4.1 (GND), U4.2 (CSB), U4.7 (GND), U5.2 (GND), U6.2 (GND), U7.4 (GND), Y1.2 (GND), C25.1, J12.2 (Pin_2)
- net +5V_BAT: now also J12.1 (Pin_1)
- net at Y1.1 (EN): now also Y1.4 (Vdd), C25.2; no longer U1.5 (PH0)
- net at Y1.3 (OUT): now also U1.5 (PH0); no longer U1.6 (PH1)
- removed net GND: C12.2, C13.2, C14.2, C15.2, C16.2, C18.2, C20.2, C21.2, C22.2, C23.2, C24.2, D1.2 (A), D2.1 (K), D5.1 (K), D6.1 (K), J1.A1 (GND), J1.A12 (GND), J1.B1 (GND), J1.B12 (GND), J1.S1 (SHIELD), J2.4 (Pin_4), J7.5 (Pin_5), LS1.N, R13.1, R2.2, R3.2, R6.1, SW1.1 (A), U1.12 (VSSA), U1.18 (VSS), U1.31 (VSS), U1.47 (VSS), U1.63 (VSS), U2.2 (GND), U3.11 (RESV_11), U3.6 (GND), U3.9 (INT2/FSYNC/CLKIN), U4.1 (GND), U4.7 (GND), U5.2 (GND), U6.2 (GND), U7.4 (GND), Y1.2 (GND), Y1.4 (Vdd)
Other:
- moved on the sheet: Y1
