File: hardware/pcb/flight_controller/flight_controller.kicad_sch (KiCad schematic)
At the start: 65 parts, among them J1 USB_C_Receptacle, J10 USART2_PINOUT, J11 I2C2_PINOUT, J12 XT_WIRE_SOLDERING_HOLES, J2 ELRS, J3 ESC1, J4 ESC1, J5 ESC1, J6 ESC1, J7 STM32_STLINK, J8 SPI3_PINOUT, J9 USART4_PINOUT, SW1 SW_SPDT, U1 STM32F722RETx, U2 USBLC6-2SC6, U3 ICM-42688-P, U4 DPS368XTSA1, U5 MP2451DJ-LF-Z, U6 AP2112K-3.3TRG1, U7 W25Q128JVSIQ, Y1 ASE-25MHz

Commit message: feat(fc): fixed buck reg caps' and resistors' value
Parts:
- removed R6: 23.7kR, symbol Device:R
- removed R7: 124kR, symbol Device:R
- added R14: 8.9kR, symbol Device:R
- added R15: 47kR, symbol Device:R
- C18: value 4.7uF -> 22uF
- C20: value 10uF -> 22uF
- J4: value ESC1 -> ESC2
- J5: value ESC1 -> ESC3
- J6: value ESC1 -> ESC4
- L1: value 4.7uH -> 6.8uH
Connections:
- net +3.3V: now also R14.1
- net +5V_BAT: now also R15.1
- net at C17.1, U5.3 (FB): now also R14.2, R15.2

Commit message: feat(esc): config buck reg to 12v
Parts:
- L1: value 6.8uH -> 10uH
Changed lines of the file:
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@@
 			)
 		)
-		(property "Value" "6.8uH"
+		(property "Value" "10uH"
 			(at 349.25 45.72 90)
 			(show_name no)
